File: KiCAD/set_board_avr/set_board_avr.kicad_sch (KiCad schematic)
At the start: 34 parts, among them J1 Conn_01x10, J2 AVR-ISP-6, Q1 Q_NPN, Q2 Q_NPN, Q3 Q_NPN, U1 ATtiny4313-S, U4 74HC14, U5 NCP1117-3.3_SOT223, Y1 ASV-xxxMHz

Commit message: working on routing
Parts:
- removed C4: 1.0uF, Capacitor_SMD:C_1206_3216Metric_Pad1.33x1.80mm_HandSolder, symbol Device:C
Changed lines of the file:
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@@
 	)
 	(junction
-		(at 232.41 39.37)
-		(diameter 0)
-		(color 0 0 0 0)
-	)
-	(junction
 		(at 219.71 95.25)
 		(diameter 0)
@@
 	(wire
 		(pts
-			(xy 219.71 39.37) (xy 219.71 72.39)
+			(xy 219.71 57.15) (xy 219.71 72.39)
 		)
 		(stroke
@@
 	(wire
 		(pts
-			(xy 219.71 39.37) (xy 232.41 39.37)
-		)
-		(stroke
-			(width 0)
-			(type default)
-		)
-	)
-	(wire
-		(pts
 			(xy 210.82 120.65) (xy 210.82 90.17)
 		)
@@
 	(wire
 		(pts
-			(xy 232.41 35.56) (xy 232.41 39.37)
-		)
-		(stroke
-			(width 0)
-			(type default)
-		)
-	)
-	(wire
-		(pts
 			(xy 195.58 82.55) (xy 219.71 82.55)
 		)
@@
 	(symbol
 		(lib_id "power:+12V")
-		(at 232.41 35.56 0)
+		(at 219.71 57.15 0)
 		(unit 1)
 		(body_style 1)
@@
 		(fields_autoplaced yes)
 		(property "Reference" "#PWR022"
-			(at 232.41 39.37 0)
+			(at 219.71 60.96 0)
 			(hide yes)
 			(show_name no)
@@
 		)
 		(property "Value" "+12V"
-			(at 232.41 30.48 0)
+			(at 219.71 52.07 0)
 			(show_name no)
 			(do_not_autoplace no)
@@
 		)
 		(property "Footprint" ""
-			(at 232.41 35.56 0)
+			(at 219.71 57.15 0)
 			(hide yes)
 			(show_name no)
@@
 		)
 		(property "Datasheet" ""
-			(at 232.41 35.56 0)
+			(at 219.71 57.15 0)
 			(hide yes)
 			(show_name no)
@@
 		)
 		(property "Description" "Power symbol creates a global label with name \"+12V\""
-			(at 232.41 35.56 0)
+			(at 219.71 57.15 0)
 			(hide yes)
 			(show_name no)
@@
 	)
 	(symbol
-		(lib_id "Device:C")
-		(at 232.41 43.18 0)
-		(unit 1)
-		(body_style 1)
-		(exclude_from_sim no)
-		(in_bom yes)
-		(on_board yes)
-		(in_pos_files yes)
-		(dnp no)
-		(fields_autoplaced yes)
-		(property "Reference" "C4"
-			(at 236.22 41.9099 0)
-			(show_name no)
-			(do_not_autoplace no)
-			(effects
-				(font
-					(size 1.27 1.27)
-				)
-				(justify left)
-			)
-		)
-		(property "Value" "1.0uF"
-			(at 236.22 44.4499 0)
-			(show_name no)
-			(do_not_autoplace no)
-			(effects
-				(font
-					(size 1.27 1.27)
-				)
-				(justify left)
-			)
-		)
-		(property "Footprint" "Capacitor_SMD:C_1206_3216Metric_Pad1.33x1.80mm_HandSolder"
-			(at 233.3752 46.99 0)
-			(hide yes)
-			(show_name no)
-			(do_not_autoplace no)
-			(effects
-				(font
-					(size 1.27 1.27)
-				)
-			)
-		)
-		(property "Datasheet" ""
-			(at 232.41 43.18 0)
-			(hide yes)
-			(show_name no)
-			(do_not_autoplace no)
-			(effects
-				(font
-					(size 1.27 1.27)
-				)
-			)
-		)
-		(property "Description" "Unpolarized capacitor"
-			(at 232.41 43.18 0)
-			(hide yes)
-			(show_name no)
-			(do_not_autoplace no)
-			(effects
-				(font
-					(size 1.27 1.27)
-				)
-			)
-		)
-		(property "Sim.Device" ""
-			(at 232.41 43.18 0)
-			(hide yes)
-			(show_name no)
-			(do_not_autoplace no)
-			(effects
-				(font
-					(size 1.27 1.27)
-				)
-			)
-		)
-		(property "Sim.Type" ""
-			(at 232.41 43.18 0)
-			(hide yes)
-			(show_name no)
-			(do_not_autoplace no)
-			(effects
-				(font
-					(size 1.27 1.27)
-				)
-			)
-		)
-		(property "CatNo" "1276-1097-1-ND"
-			(at 232.41 43.18 0)
-			(hide yes)
-			(show_name no)
-			(do_not_autoplace no)
-			(effects
-				(font
-					(size 1.27 1.27)
-				)
-			)
-		)
-		(property "MfgNo" "CL31B105KAHNNNE"
-			(at 232.41 43.18 0)
-			(hide yes)
-			(show_name no)
-			(do_not_autoplace no)
-			(effects
-				(font
-					(size 1.27 1.27)
-				)
-			)
-		)
-		(pin "1"
-		)
-		(pin "2"
-		)
-		(instances
-			(project "set_board_avr"
-				(path "/c1980bc9-cc73-4b12-bf5e-a245c9009914"
-					(reference "C4")
-					(unit 1)
-				)
-			)
-		)
-	)
-	(symbol
 		(lib_id "Connector:AVR-ISP-6")
 		(at 39.37 113.03 0)
@@
 					(unit 1)
 				)
-			)
-		)
-	)
-	(symbol
-		(lib_id "set_board-rescue:GND-power")
-		(at 232.41 46.99 0)
-		(unit 1)
-		(body_style 1)
-		(exclude_from_sim no)
-		(in_bom yes)
-		(on_board yes)
-		(in_pos_files yes)
-		(dnp no)
-		(property "Reference" "#PWR020"
-			(at 232.41 53.34 0)
-			(hide yes)
-			(show_name no)
-			(do_not_autoplace no)
-			(effects
-				(font
-					(size 1.27 1.27)
-				)
-			)
-		)
-		(property "Value" "GND"
-			(at 236.22 48.26 0)
-			(show_name no)
-			(do_not_autoplace no)
-			(effects
-				(font
-					(size 1.27 1.27)
-				)
-			)
-		)
-		(property "Footprint" ""
-			(at 232.41 46.99 0)
-			(hide yes)
-			(show_name no)
-			(do_not_autoplace no)
-			(effects
-				(font
-					(size 1.27 1.27)
-				)
-			)
-		)
-		(property "Datasheet" ""
-			(at 232.41 46.99 0)
-			(hide yes)
-			(show_name no)
-			(do_not_autoplace no)
-			(effects
-				(font
-					(size 1.27 1.27)
-				)
-			)
-		)
-		(property "Description" ""
-			(at 232.41 46.99 0)
-			(hide yes)
-			(show_name no)
-			(do_not_autoplace no)
-			(effects
-				(font
-					(size 1.27 1.27)
-				)
-			)
-		)
-		(pin "1"
-		)
-		(instances
-			(project "set_board_avr"
-				(path "/c1980bc9-cc73-4b12-bf5e-a245c9009914"
-					(reference "#PWR020")
-					(unit 1)
-				)

Commit message: update for WWVB
Parts:
- removed C7: 0.1uF, Capacitor_SMD:C_1206_3216Metric_Pad1.33x1.80mm_HandSolder, symbol Device:C
- removed U2: (no value), my_wifi:ESP8266_Wifi_module, symbol my_wifi:esp8266_wifi
- removed Y1: ASV-xxxMHz, Oscillator:Oscillator_SMD_Abracon_ASV-4Pin_7.0x5.1mm, symbol Oscillator:ASV-xxxMHz
- added J3: RJ45, my_RJ45:Metz_AJT65B8813, symbol Connector:RJ45
- added R15, R16, R17: 1k, Resistor_SMD:R_1206_3216Metric_Pad1.30x1.75mm_HandSolder, symbol Device:R_US
- added R18: 100, Resistor_SMD:R_1206_3216Metric_Pad1.30x1.75mm_HandSolder, symbol Device:R_US
- C3: value 470uF -> 100uF; footprint Capacitor_THT:CP_Radial_D8.0mm_P3.50mm -> (none); CatNo 1189-3712-1-ND -> 399-ESH107M6R3AC3AA-ND; MfgNo 16ZLH470MEFCT78X11.5 -> (none)
Connections:
- net +3.3V: now also R18.1; no longer C3.1
- net GND: now also J3.2, J3.5, J3.6, J3.8, J3.S1 (GND), J3.S2 (GND)
- net WWVB: now reaches U1.2 (PD0)
- net WWVB: now also J3.3, R15.2
- net SPARE1: now reaches U1.9 (PD5)
- net SPARE1: now also J3.7, R17.2
- net SPARE0: now reaches U1.3 (PD1)
- net SPARE0: now also J3.4, R16.2
- new net: C3.1, J3.1, R15.1, R16.1, R17.1, R18.2

Commit message: finish place/route on set_board_avr
Parts:
- C3: footprint (none) -> Capacitor_THT:CP_Radial_D5.0mm_P2.00mm; CatNo 399-ESH107M6R3AC3AA-ND -> ESH107M010AC3AA
Changed lines of the file:
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@@
 			)
 		)
-		(property "Footprint" ""
+		(property "Footprint" "Capacitor_THT:CP_Radial_D5.0mm_P2.00mm"
 			(at 196.5452 153.67 0)
 			(hide yes)
@@
 			)
 		)
-		(property "CatNo" "399-ESH107M6R3AC3AA-ND"
+		(property "CatNo" "ESH107M010AC3AA"
 			(at 210.566 153.924 0)
 			(show_name no)
