File: KiCAD/set_board_avr/set_board_avr.kicad_pcb (KiCad board)
At the start: 2 copper layers, 197.5 x 17.8 mm, 35 parts, among them J1 Conn_01x10, J2 AVR-ISP-6, J3 RJ45, Q1 Q_NPN, Q2 Q_NPN, Q3 Q_NPN, U1 ATtiny4313-S, U4 74HC14, U5 NCP1117-3.3_SOT223

Commit message: maybe add BAV99 protection diodes?
Parts:
- added D4: BAV99, Package_TO_SOT_SMD:SOT-23, B.Cu at (116.9, 54.0)
- added D5: BAV99, Package_TO_SOT_SMD:SOT-23, B.Cu at (116.9, 58.5)
- added D6: BAV99, Package_TO_SOT_SMD:SOT-23, B.Cu at (116.9, 62.9)
- added D7: BAV99, Package_TO_SOT_SMD:SOT-23, B.Cu at (116.9, 67.4)
Routing:
- net GND: vias 22 -> 26
